File: Hardware/Deej_ESP_PCB/Deej_ESP_PCB.kicad_sch (KiCad schematic)
At the start: 149 parts, among them J1 USB_C_Receptacle_USB2.0_16P, J2 UART Header, P1 10K, P2 10K, P3 10K, P4 10K, P5 10K, P6 10K, SW1 SW_Push, SW2 SW_Push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

Commit message: -Trace routing 'done' ... until I find another issue -Fixing DRC errors and warnings
Parts:
- H1, H3, H5, H7, H9: value ~ -> (none)
